Commit message: ekf works

File: description/robot_core.xacro (robot description, xacro)
@@ -39,5 +39,5 @@
 			</geometry>
 		</collision>>
-		<xacro:inertial_box mass="0.5" x="0.692" y="0.304" z="0.296">
+		<xacro:inertial_box mass="0.5" x="0.692" y="0.304" z="0.3">
 			<origin xyz="0 0 .11" rpy="0 0 0"/>
 		</xacro:inertial_box>
@@ -52,5 +52,5 @@
 		<child link="rear_left_wheel"/>
 		<!-- physically rotating cylinder & placing it correctly -->
-		<origin xyz="-.296 .218 .17" rpy="-${pi/2} 0 0"/>
+		<origin xyz="-.3 .21 .17" rpy="-${pi/2} 0 0"/>
 		<!-- rotation axis -->
 		<axis xyz="0 0 1"/>
@@ -81,5 +81,5 @@
 		<child link="front_left_wheel"/>
 		<!-- physically rotating cylinder & placing it correctly -->
-		<origin xyz=".296 .218 .17" rpy="-${pi/2} 0 0"/>
+		<origin xyz=".3 .21 .17" rpy="-${pi/2} 0 0"/>
 		<!-- rotation axis -->
 		<axis xyz="0 0 1"/>
@@ -110,5 +110,5 @@
 		<child link="rear_right_wheel"/>
 		<!-- physically rotating cylinder & placing it correctly -->
-		<origin xyz="-.296 -.218 .17" rpy="-${pi/2} 0 0"/>
+		<origin xyz="-.3 -.21 .17" rpy="-${pi/2} 0 0"/>
 		<!-- rotation axis -->
 		<axis xyz="0 0 1"/>
@@ -139,5 +139,5 @@
 		<child link="front_right_wheel"/>
 		<!-- physically rotating cylinder & placing it correctly -->
-		<origin xyz=".296 -.218 .17" rpy="-${pi/2} 0 0"/>
+		<origin xyz=".3 -.21 .17" rpy="-${pi/2} 0 0"/>
 		<!-- rotation axis -->
 		<axis xyz="0 0 1"/>
@@ -159,4 +159,28 @@
 		</xacro:inertial_cylinder>
 	</link>
+    <joint name="camera_joint" type="fixed">
+        <parent link="base_link"/>
+        <child link="camera_frame"/>
+        <origin xyz=".39 0 .36" rpy="0 0 0"/>
+    </joint>
+    <link name="camera_frame">
+        <visual>
+            <geometry>
+                <box size="0.1 0.4 0.1"/>
+            </geometry>
+        </visual>
+    </link>
+    <joint name="gps_joint" type="fixed">
+        <parent link="base_link"/>
+        <child link="gps_frame"/>
+        <origin xyz=".33 0 1.03" rpy="0 0 0"/>
+    </joint>
+    <link name="gps_frame">
+        <visual>
+            <geometry>
+                <box size="0.1 0.1 0.1"/>
+            </geometry>
+        </visual>
+    </link>
 	<gazebo reference="front_right_wheel">
 		<material>Gazebo/Blue</material>

File: description/ros2_control.xacro (robot description, xacro)
@@ -39,13 +39,22 @@
     <ros2_control name="OSCAR" type="system">
         <hardware>
-		    <plugin>oscar_hardware_intf/OscarHardwareIntf</plugin>
+		    <plugin>oscar_hardware_intf/OscarSimulationIntf</plugin>
+            <!-->
             <param name="encoder_cpr">16000</param>
             <param name="micro_run_freq">100</param>
-            <param name="serial_port">/dev/ttyUSB0</param>
+            <param name="serial_port">/dev/ttyUSB0</param><-->
         </hardware>
         <joint name="front_left_wheel_joint">
             <command_interface name="velocity">
-                <param name="min">-2</param>
-                <param name="max">2</param>
+                <param name="min">-10</param>
+                <param name="max">10</param>
+            </command_interface>
+            <state_interface name="position"/>
+            <state_interface name="velocity"/>
+        </joint>
+        <joint name="front_right_wheel_joint">
+            <command_interface name="velocity">
+                <param name="min">-10</param>
+                <param name="max">10</param>
             </command_interface>
             <state_interface name="position"/>
@@ -54,14 +63,6 @@
         <joint name="rear_left_wheel_joint">
             <command_interface name="velocity">
-                <param name="min">-2</param>
-                <param name="max">2</param>
-            </command_interface>
-            <state_interface name="position"/>
-            <state_interface name="velocity"/>
-        </joint>
-        <joint name="front_right_wheel_joint">
-            <command_interface name="velocity">
-                <param name="min">-2</param>
-                <param name="max">2</param>
+                <param name="min">-10</param>
+                <param name="max">10</param>
             </command_interface>
             <state_interface name="position"/>
@@ -70,6 +71,6 @@
         <joint name="rear_right_wheel_joint">
             <command_interface name="velocity">
-                <param name="min">-2</param>
-                <param name="max">2</param>
+                <param name="min">-10</param>
+                <param name="max">10</param>
             </command_interface>
             <state_interface name="position"/>
