Commit message: ros2 control fixes

File: description/real/ros2_control.xacro (robot description, xacro)
@@ -16,5 +16,5 @@
             <state_interface name="velocity"/>
         </joint>
-        <joint name="front_right_wheel_joint">
+        <joint name="rear_left_wheel_joint">
             <command_interface name="velocity">
                 <param name="min">-10</param>
@@ -24,5 +24,5 @@
             <state_interface name="velocity"/>
         </joint>
-        <joint name="rear_left_wheel_joint">
+        <joint name="front_right_wheel_joint">
             <command_interface name="velocity">
                 <param name="min">-10</param>
