Commit message: ekf, gps, zed configs for jetson

File: description/real/robot_core.xacro (robot description, xacro)
@@ -1,5 +1,5 @@
 <?xml version="1.0"?>
 <robot xmlns:xacro="http://www.ros.org/wiki/xacro"  name="robot">
-	<xacro:include filename="inertial_macros.xacro"/>
+	<xacro:include filename="../inertial_macros.xacro"/>
 	<material name="white">
 		<color rgba="1 1 1 1"/>
@@ -159,16 +159,4 @@
 		</xacro:inertial_cylinder>
 	</link>
-    <joint name="camera_joint" type="fixed">
-        <parent link="base_link"/>
-        <child link="camera_frame"/>
-        <origin xyz=".39 0 .36" rpy="0 0 0"/>
-    </joint>
-    <link name="camera_frame">
-        <visual>
-            <geometry>
-                <box size="0.1 0.4 0.1"/>
-            </geometry>
-        </visual>
-    </link>
     <joint name="gps_joint" type="fixed">
         <parent link="base_link"/>

File: description/sim/ros2_control.xacro (robot description, xacro)
@@ -80,5 +80,5 @@
     <gazebo>
         <plugin name="gazebo_ros2_control" filename="libgazebo_ros2_control.so">
-            <parameters>$(find oscar_ros)/config/my_controllers.yaml</parameters>
+            <parameters>$(find oscar_ros)/config/sim/my_controllers.yaml</parameters>
         </plugin>
     </gazebo>

Commit message: septentrio gps config

File: description/real/robot_core.xacro (robot description, xacro)
@@ -171,4 +171,16 @@
         </visual>
     </link>
+    <joint name="aux1_joint" type="fixed">
+        <parent link="base_link"/>
+        <child link="aux1_frame"/>
+        <origin xyz="-.33 0 1.03" rpy="0 0 0"/>
+    </joint>
+    <link name="aux1_frame">
+        <visual>
+            <geometry>
+                <box size="0.1 0.1 0.1"/>
+            </geometry>
+        </visual>
+    </link>
 	<gazebo reference="front_right_wheel">
 		<material>Gazebo/Blue</material>

Commit message: Re-tuned global UKF, added BNO055 configs

File: description/real/robot_core.xacro (robot description, xacro)
@@ -183,4 +183,16 @@
         </visual>
     </link>
+    <joint name="bno055_joint" type="fixed">
+        <parent link="base_link"/>
+        <child link="bno055"/>
+        <origin xyz="-0.05 0 0.17" rpy="0 0 0"/>
+    </joint>
+    <link name="bno055">
+        <visual>
+            <geometry>
+                <box size="0.1 0.1 0.1"/>
+            </geometry>
+        </visual>
+    </link>
 	<gazebo reference="front_right_wheel">
 		<material>Gazebo/Blue</material>
